Commit message: migration

File: urdf/robot.urdf.xacro (robot description, xacro)
@@ -74,25 +74,34 @@
         <origin xyz="0.2 0 -0.075"/> </joint>
     <gazebo>
-        <plugin name="diff_drive" filename="libgazebo_ros_diff_drive.so">
-            <update_rate>50</update_rate>
+        <!-- Actuation only: its odometry/tf go to unbridged topics -->
+        <plugin filename="gz-sim-diff-drive-system" name="gz::sim::systems::DiffDrive">
             <left_joint>left_joint</left_joint>
             <right_joint>right_joint</right_joint>
             <wheel_separation>0.34</wheel_separation>
-            <wheel_diameter>0.1</wheel_diameter>
-            <max_wheel_torque>20</max_wheel_torque>
-            <max_wheel_acceleration>1.0</max_wheel_acceleration>
-            <publish_odom>true</publish_odom>
-            <publish_odom_tf>true</publish_odom_tf>
-            <publish_wheel_tf>true</publish_wheel_tf>
-             <command_topic>cmd_vel</command_topic>
-            <odometry_frame>odom</odometry_frame>
+            <wheel_radius>0.05</wheel_radius>
+            <max_linear_acceleration>1.0</max_linear_acceleration>
+            <topic>/cmd_vel</topic>
+            <odom_topic>/diff_drive/odom</odom_topic>
+            <tf_topic>/diff_drive/tf</tf_topic>
+            <frame_id>odom</frame_id>
+            <child_frame_id>base_link</child_frame_id>
+        </plugin>
+        <!-- Ground-truth odometry (like gazebo_ros_p3d), stays correct after teleport resets -->
+        <plugin filename="gz-sim-odometry-publisher-system" name="gz::sim::systems::OdometryPublisher">
+            <odom_frame>odom</odom_frame>
             <robot_base_frame>base_link</robot_base_frame>
+            <odom_topic>/odom</odom_topic>
+            <tf_topic>/tf</tf_topic>
+            <odom_publish_frequency>50</odom_publish_frequency>
+            <dimensions>2</dimensions>
         </plugin>
-        <plugin name="gazebo_ros_p3d" filename="libgazebo_ros_p3d.so">
-             </plugin>
+        <plugin filename="gz-sim-joint-state-publisher-system" name="gz::sim::systems::JointStatePublisher">
+            <topic>/joint_states</topic>
+        </plugin>
     </gazebo>
-    <gazebo reference="base_link"><material>Gazebo/Blue</material></gazebo>
-    <gazebo reference="left_wheel"><material>Gazebo/Black</material></gazebo>
-    <gazebo reference="right_wheel"><material>Gazebo/Black</material></gazebo>
+    <gazebo reference="caster_wheel">
+        <mu1>0.01</mu1>
+        <mu2>0.01</mu2>
+    </gazebo>
     <link name="lidar_link">
         <visual>
@@ -114,9 +123,11 @@
     </joint>
     <gazebo reference="lidar_link">
-        <sensor name="lidar" type="ray">
+        <sensor name="lidar" type="gpu_lidar">
             <always_on>true</always_on>
             <visualize>true</visualize>
             <update_rate>10</update_rate>
-            <ray>
+            <topic>/scan</topic>
+            <gz_frame_id>lidar_link</gz_frame_id>
+            <lidar>
                 <scan>
                     <horizontal>
@@ -126,4 +137,10 @@
                         <max_angle>6.280000</max_angle>
                     </horizontal>
+                    <vertical>
+                        <samples>1</samples>
+                        <resolution>1</resolution>
+                        <min_angle>0</min_angle>
+                        <max_angle>0</max_angle>
+                    </vertical>
                 </scan>
                 <range>
@@ -132,12 +149,5 @@
                     <resolution>0.015000</resolution>
                 </range>
-            </ray>
-            <plugin name="scan" filename="libgazebo_ros_ray_sensor.so">
-                <ros>
-                    <remapping>~/out:=scan</remapping>
-                </ros>
-                <output_type>sensor_msgs/LaserScan</output_type>
-                <frame_name>lidar_link</frame_name>
-            </plugin>
+            </lidar>
         </sensor>
     </gazebo>
